File: DC-DC 12-450V.kicad_pcb (KiCad board)
At the start: 2 copper layers, 85 x 50 mm, 44 parts, among them J1 12V input, J2 HV output, Q1 IRF3205, Q2 S8050, U1 UC3843_DIP8

Commit message: Add files via upload
Parts:
- removed TP5: e, TestPoint:TestPoint_THTPad_D3.0mm_Drill1.5mm
- added PAD9: , TestPoint:TestPoint_THTPad_D3.0mm_Drill1.5mm, F.Cu at (160.8, 81.2)
- D2: value FES8JT -> MUR860
- PAD4: renamed from TP5; value e -> (none)
- R11: value 15mR -> 0.015R
- U1: value UC3843_DIP8 -> UC3843BN_DIP8
- renumbered TP1 to PAD1, TP5 to PAD10, TP5 to PAD11, TP1 to PAD12, TP5 to PAD2, TP5 to PAD3, TP5 to PAD5, TP2 to PAD6, TP2 to PAD7, TP5 to PAD8
Connections:
- PAD10 pad 10: GND -> Net-(D2-K)
- PAD11 pad 11: GND -> Net-(D2-K)
Routing:
- net Net-(D2-K): track 31.1 -> 44.2 mm
- net GND: track 140.6 -> 147.4 mm

Commit message: Add files via upload
Parts:
- turned C8 to 90 degrees
Connections:
- PAD1 pad 1: Net-(Q1-D) -> +12V
- PAD12 pad 12: (no net) -> Net-(D2-A)
- PAD6 pad 6: (no net) -> Net-(Q1-D)
- PAD7 pad 7: (no net) -> +12V
Changed lines of the file:
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@@
 			(layers "*.Cu" "*.Mask")
 			(remove_unused_layers no)
+			(net 10 "Net-(D2-A)")
 		)
 		(embedded_fonts no)
@@
 	(footprint "Capacitor_SMD:C_1206_3216Metric"
 		(layer "F.Cu")
-		(at 126.5 80 -90)
+		(at 126.5 80 90)
 		(descr "Capacitor SMD 1206 (3216 Metric), square (rectangular) end terminal, IPC_7351 nominal, (Body size source: IPC-SM-782 page 76, https://www.pcb-3d.com/wordpress/wp-content/uploads/ipc-sm-782a_amendment_1_and_2.pdf), generated with kicad-footprint-generator")
 		(tags "capacitor")
@@
 		)
 		(property "Datasheet" "~"
-			(at 0 0 270)
+			(at 0 0 90)
 			(unlocked yes)
 			(layer "F.Fab")
@@
 		)
 		(property "Description" "Unpolarized capacitor, small symbol"
-			(at 0 0 270)
+			(at 0 0 90)
 			(unlocked yes)
 			(layer "F.Fab")
@@
 		(attr smd)
 		(fp_line
-			(start -0.711252 0.91)
-			(end 0.711252 0.91)
+			(start -0.711252 -0.91)
+			(end 0.711252 -0.91)
 			(stroke
 				(width 0.12)
@@
 		)
 		(fp_line
-			(start -0.711252 -0.91)
-			(end 0.711252 -0.91)
+			(start -0.711252 0.91)
+			(end 0.711252 0.91)
 			(stroke
 				(width 0.12)
@@
 		)
 		(fp_line
-			(start -2.3 1.15)
-			(end -2.3 -1.15)
+			(start 2.3 -1.15)
+			(end 2.3 1.15)
 			(stroke
 				(width 0.05)
@@
 		)
 		(fp_line
-			(start 2.3 1.15)
-			(end -2.3 1.15)
+			(start -2.3 -1.15)
+			(end 2.3 -1.15)
 			(stroke
 				(width 0.05)
@@
 		)
 		(fp_line
-			(start -2.3 -1.15)
-			(end 2.3 -1.15)
+			(start 2.3 1.15)
+			(end -2.3 1.15)
 			(stroke
 				(width 0.05)
@@
 		)
 		(fp_line
-			(start 2.3 -1.15)
-			(end 2.3 1.15)
+			(start -2.3 1.15)
+			(end -2.3 -1.15)
 			(stroke
 				(width 0.05)
@@
 		)
 		(fp_line
-			(start -1.6 0.8)
-			(end -1.6 -0.8)
+			(start 1.6 -0.8)
+			(end 1.6 0.8)
 			(stroke
 				(width 0.1)
@@
 		)
 		(fp_line
-			(start 1.6 0.8)
-			(end -1.6 0.8)
+			(start -1.6 -0.8)
+			(end 1.6 -0.8)
 			(stroke
 				(width 0.1)
@@
 		)
 		(fp_line
-			(start -1.6 -0.8)
-			(end 1.6 -0.8)
+			(start 1.6 0.8)
+			(end -1.6 0.8)
 			(stroke
 				(width 0.1)
@@
 		)
 		(fp_line
-			(start 1.6 -0.8)
-			(end 1.6 0.8)
+			(start -1.6 0.8)
+			(end -1.6 -0.8)
 			(stroke
 				(width 0.1)
@@
 		)
 		(pad "1" smd roundrect
-			(at -1.475 0 270)
+			(at -1.475 0 90)
 			(size 1.15 1.8)
 			(layers "F.Cu" "F.Mask" "F.Paste")
@@
 		)
 		(pad "2" smd roundrect
-			(at 1.475 0 270)
+			(at 1.475 0 90)
 			(size 1.15 1.8)
 			(layers "F.Cu" "F.Mask" "F.Paste")
@@
 			(layers "*.Cu" "*.Mask")
 			(remove_unused_layers no)
-			(net 12 "Net-(Q1-D)")
+			(net 9 "+12V")
 			(pinfunction "1")
 			(pintype "passive")
@@
 			(layers "*.Cu" "*.Mask")
 			(remove_unused_layers no)
+			(net 9 "+12V")
 		)
 		(embedded_fonts no)
@@
 			(layers "*.Cu" "*.Mask")
 			(remove_unused_layers no)
+			(net 12 "Net-(Q1-D)")
 		)
 		(embedded_fonts no)

Commit message: Add files via upload
Parts:
- PAD1: value Q1-D -> +12V
- R11: footprint Resistor_SMD:R_2816_7142Metric -> Resistor_SMD:R_2512_6332Metric
- moved D1 1.00 mm to (106.5, 99.5), turned to 90 degrees
- moved R12 0.75 mm to (167.2, 61.8), turned to 180 degrees
- turned D3 to 180 degrees
Connections:
- net Net-(Q1-S) renamed /Q1-S
- D2 pad 2: Net-(D2-A) -> /D2-A
- Q1 pad 2: Net-(Q1-D) -> /Q1-D
Routing:
- net GND: track 147.4 -> 144.0 mm, vias 9 -> 21
- net +12V: track 109.5 -> 108.3 mm
- net Net-(D3-A): track 3.51 -> 2.40 mm
- added copper zone on F.Cu, net +12V
- added copper zone on F.Cu, net /Q1-S
