File: DC-DC 12-450V.kicad_pcb (KiCad board)
At the start: 2 copper layers, 85 x 50 mm, 46 parts, among them J1 12V input, J2 HV output, Q1 IRF3205, Q2 S8050, U1 UC3843BN_DIP8

Commit message: Add files via upload
Parts:
- RV1: footprint Potentiometer_THT:Potentiometer_Bourns_3266Y_Vertical -> Potentiometer_THT:Potentiometer_Bourns_3296W_Vertical
Connections:
- Q2 pad 1: unconnected-(Q2-B-Pad1) -> Net-(Q2-B)
- R10 pad 1: Net-(R10-Pad1) -> Net-(Q2-B)
- RV1 pad 2: Net-(R10-Pad1) -> Net-(Q2-B)
- RV1 pad 3: Net-(R10-Pad1) -> Net-(Q2-B)
Routing:
- net Net-(Q2-B): track 0.00 -> 14.7 mm
- net (no net): track 14.7 -> 0.00 mm
Changed lines of the file:
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@@
 	(net 20 "/Q1-S")
 	(net 21 "/VCC")
-	(net 22 "unconnected-(Q2-B-Pad1)")
-	(net 23 "Net-(R10-Pad1)")
+	(net 22 "Net-(Q2-B)")
 	(footprint "Capacitor_THT:CP_Radial_D10.0mm_P5.00mm"
 		(layer "F.Cu")
@@
 			(layers "F.Cu" "F.Mask" "F.Paste")
 			(roundrect_rratio 0.222222)
-			(net 23 "Net-(R10-Pad1)")
+			(net 22 "Net-(Q2-B)")
 			(pintype "passive")
 		)
@@
 			(layers "F.Cu" "F.Mask" "F.Paste")
 			(roundrect_rratio 0.25)
-			(net 22 "unconnected-(Q2-B-Pad1)")
+			(net 22 "Net-(Q2-B)")
 			(pinfunction "B")
 			(pintype "input")
@@
 		)
 	)
-	(footprint "Potentiometer_THT:Potentiometer_Bourns_3266Y_Vertical"
+	(footprint "Potentiometer_THT:Potentiometer_Bourns_3296W_Vertical"
 		(layer "F.Cu")
 		(at 107.5 69.71 90)
-		(descr "Potentiometer, vertical, Bourns 3266Y, https://www.bourns.com/docs/Product-Datasheets/3266.pdf")
-		(tags "Potentiometer vertical Bourns 3266Y")
+		(descr "Potentiometer, vertical, Bourns 3296W, https://www.bourns.com/pdfs/3296.pdf")
+		(tags "Potentiometer vertical Bourns 3296W")
 		(property "Reference" "RV1"
-			(at -2.525 3.5 90)
+			(at -2.54 -3.66 90)
 			(layer "F.SilkS")
 			(effects
@@
 		)
 		(property "Value" "5K"
-			(at -2.54 3.59 90)
+			(at -2.54 3.67 90)
 			(layer "F.Fab")
-			(hide yes)
 			(effects
 				(font
@@
 		(attr through_hole exclude_from_bom)
 		(fp_line
-			(start 0.935 -2.28)
-			(end 0.935 -0.494)
-			(stroke
-				(width 0.12)
-				(type solid)
-			)
-			(layer "F.SilkS")
-		)
-		(fp_line
-			(start -6.015 -2.28)
-			(end 0.935 -2.28)
+			(start 2.345 -2.53)
+			(end 2.345 2.54)
 			(stroke
 				(width 0.12)
@@
 		)
 		(fp_line
-			(start -6.015 -2.28)
-			(end -6.015 -0.494)
+			(start -7.425 -2.53)
+			(end 2.345 -2.53)
 			(stroke
 				(width 0.12)
@@
 		)
 		(fp_line
-			(start 0.935 0.496)
-			(end 0.935 2.46)
+			(start -7.425 -2.53)
+			(end -7.425 2.54)
 			(stroke
 				(width 0.12)
@@
 		)
 		(fp_line
-			(start -6.015 0.496)
-			(end -6.015 2.46)
+			(start -7.425 2.54)
+			(end 2.345 2.54)
 			(stroke
 				(width 0.12)
@@
 		)
 		(fp_line
-			(start -6.015 2.46)
-			(end 0.935 2.46)
-			(stroke
-				(width 0.12)
-				(type solid)
-			)
-			(layer "F.SilkS")
-		)
-		(fp_line
-			(start 1.1 -2.45)
-			(end -6.15 -2.45)
+			(start 2.5 -2.7)
+			(end -7.6 -2.7)
 			(stroke
 				(width 0.05)
@@
 		)
 		(fp_line
-			(start -6.15 -2.45)
-			(end -6.15 2.6)
+			(start -7.6 -2.7)
+			(end -7.6 2.7)
 			(stroke
 				(width 0.05)
@@
 		)
 		(fp_line
-			(start 1.1 2.6)
-			(end 1.1 -2.45)
+			(start 2.5 2.7)
+			(end 2.5 -2.7)
 			(stroke
 				(width 0.05)
@@
 		)
 		(fp_line
-			(start -6.15 2.6)
-			(end 1.1 2.6)
+			(start -7.6 2.7)
+			(end 2.5 2.7)
 			(stroke
 				(width 0.05)
@@
 		)
 		(fp_line
-			(start 0.815 -2.16)
-			(end -5.895 -2.16)
+			(start 2.225 -2.41)
+			(end -7.305 -2.41)
 			(stroke
 				(width 0.1)
@@
 		)
 		(fp_line
-			(start -5.895 -2.16)
-			(end -5.895 2.34)
+			(start -7.305 -2.41)
+			(end -7.305 2.42)
 			(stroke
 				(width 0.1)
@@
 		)
 		(fp_line
-			(start -0.405 1.952)
-			(end -0.404 0.189)
+			(start 0.955 2.235)
+			(end 0.956 0.066)
 			(stroke
 				(width 0.1)
@@
 		)
 		(fp_line
-			(start -0.405 1.952)
-			(end -0.404 0.189)
+			(start 0.955 2.235)
+			(end 0.956 0.066)
 			(stroke
 				(width 0.1)
@@
 		)
 		(fp_line
-			(start 0.815 2.34)
-			(end 0.815 -2.16)
+			(start 2.225 2.42)
+			(end 2.225 -2.41)
 			(stroke
 				(width 0.1)
@@
 		)
 		(fp_line
-			(start -5.895 2.34)
-			(end 0.815 2.34)
+			(start -7.305 2.42)
+			(end 2.225 2.42)
 			(stroke
 				(width 0.1)
@@
 		)
 		(fp_circle
-			(center -0.405 1.07)
-			(end 0.485 1.07)
+			(center 0.955 1.15)
+			(end 2.05 1.15)
 			(stroke
 				(width 0.1)
@@
 		)
 		(fp_text user "${REFERENCE}"
-			(at -3.15 0.09 90)
+			(at -3.175 0.005 90)
 			(layer "F.Fab")
 			(effects
 				(font
-					(size 0.92 0.92)
+					(size 1 1)
 					(thickness 0.15)
 				)
@@
 			(layers "*.Cu" "*.Mask")
 			(remove_unused_layers no)
-			(net 23 "Net-(R10-Pad1)")
+			(net 22 "Net-(Q2-B)")
 			(pinfunction "2")
 			(pintype "passive")
@@
 			(layers "*.Cu" "*.Mask")
 			(remove_unused_layers no)
-			(net 23 "Net-(R10-Pad1)")
+			(net 22 "Net-(Q2-B)")
 			(pinfunction "3")
 			(pintype "passive")
 		)
 		(embedded_fonts no)
-		(model "${KICAD9_3DMODEL_DIR}/Potentiometer_THT.3dshapes/Potentiometer_Bourns_3266Y_Vertical.wrl"
+		(model "${KICAD9_3DMODEL_DIR}/Potentiometer_THT.3dshapes/Potentiometer_Bourns_3296W_Vertical.wrl"
 			(offset
 				(xyz 0 0 0)
@@
 	)
 	(segment
-		(start 101.432936 74.7125)
-		(end 107.4225 74.7125)
-		(width 0.4)
-		(layer "F.Cu")
-		(net 0)
-	)
-	(segment
-		(start 107.6025 74.6875)
-		(end 107.5 74.79)
-		(width 0.2)
-		(layer "F.Cu")
-		(net 0)
-	)
-	(segment
-		(start 113.55 74.6875)
-		(end 107.6025 74.6875)
-		(width 0.4)
-		(layer "F.Cu")
-		(net 0)
-	)
-	(segment
-		(start 107.4225 74.7125)
-		(end 107.5 74.79)
-		(width 0.2)
-		(layer "F.Cu")
-		(net 0)
-	)
-	(segment
-		(start 107.5 72.25)
-		(end 107.5 74.79)
-		(width 0.4)
-		(layer "F.Cu")
-		(net 0)
-	)
-	(segment
 		(start 112.54 85.54)
 		(end 112.25 85.25)
@@
 		(net 21)
 	)
+	(segment
+		(start 101.432936 74.7125)
+		(end 107.4225 74.7125)
+		(width 0.4)
+		(layer "F.Cu")
+		(net 22)
+	)
+	(segment
+		(start 107.6025 74.6875)
+		(end 107.5 74.79)
+		(width 0.2)
+		(layer "F.Cu")
+		(net 22)
+	)
+	(segment
+		(start 113.55 74.6875)
+		(end 107.6025 74.6875)
+		(width 0.4)
+		(layer "F.Cu")
+		(net 22)
+	)
+	(segment
+		(start 107.4225 74.7125)
+		(end 107.5 74.79)
+		(width 0.2)
+		(layer "F.Cu")
+		(net 22)
+	)
+	(segment
+		(start 107.5 72.25)
+		(end 107.5 74.79)
+		(width 0.4)
+		(layer "F.Cu")
+		(net 22)
+	)
 	(zone

Commit message: Add files via upload
Parts:
- removed D4: PESD12VL1BA, Diode_SMD:D_SOD-323
- removed PAD4: , TestPoint:TestPoint_THTPad_D3.0mm_Drill1.5mm
- added C9: 100u/35V, Capacitor_THT:CP_Radial_D7.5mm_P2.50mm, F.Cu at (120.2, 66.0)
- added JP1: SolderJumper_2_Open, Jumper:SolderJumper-2_P1.3mm_Open_Pad1.0x1.5mm, F.Cu at (141.0, 64.7)
- added PAD9: , TestPoint:TestPoint_THTPad_D3.0mm_Drill1.5mm, F.Cu at (135.8, 81.2)
- C7: value 1500u/16V -> 1000u/35V
- D2: value MUR860 -> UF5407-8; footprint Package_TO_SOT_THT:TO-220-2_Vertical -> Diode_THT:D_DO-201AD_P15.24mm_Horizontal
- F2: value 1.5A/13.2V -> 1.5A/24V; footprint Fuse:Fuse_1206_3216Metric_Pad1.42x1.75mm_HandSolder -> Fuse:Fuse_1812_4532Metric_Pad1.30x3.40mm_HandSolder
- J1: value 12V input -> 12~24V input
- R12: value 1K -> 2K2
- moved R2 17.8 mm to (116.5, 94.0), turned to 180 degrees
- moved R3 10.2 mm to (116.5, 97.5), turned to 180 degrees
- moved R9 7.85 mm to (167.5, 83.0), turned to 90 degrees
- moved J1 6.46 mm to (180.5, 79.8)
- moved C3 5.76 mm to (108.0, 93.8), turned to 0 degrees
- moved RV1 5.08 mm to (107.5, 74.8), turned to -90 degrees
- moved D2 4.35 mm to (171.9, 104.8)
- moved C8 4.25 mm to (126.8, 80.2)
- moved D1 3.29 mm to (109.8, 100.0), turned to 0 degrees
- moved F2 3.18 mm to (131.8, 87.8), turned to 90 degrees
- moved R8 3.01 mm to (171.8, 83.0)
- moved R10 2.72 mm to (102.5, 70.8)
Connections:
- C7 pad 1: +12V -> +12~24V
- D2 pad 2: /D2-A -> Net-(D2-A)
- F1 pad 1: +12V -> +12~24V
- F2 pad 1: +12V -> +12~24V
- PAD1 pad 1: +12V -> (no net)
- PAD10 pad 10: Net-(D2-K) -> (no net)
- PAD11 pad 11: Net-(D2-K) -> (no net)
- PAD2 pad 2: +12V -> +12~24V
- PAD3 pad 3: +12V -> (no net)
- PAD5 pad 5: Net-(Q1-D) -> /Q1-D
- PAD6 pad 6: Net-(Q1-D) -> /Q1-D
- PAD7 pad 7: +12V -> +12~24V
- PAD8 pad 8: +12V -> +12~24V
- R12 pad 2: +12V -> +12~24V
Routing:
- net +12V: track 73.2 -> 0.00 mm
- net +12~24V: track 0.00 -> 70.5 mm
- net GND: track 144.3 -> 97.9 mm, vias 48 -> 68
- net Net-(R9-Pad1): track 64.1 -> 110.2 mm, vias 2 -> 0
- net Net-(D2-K): track 44.2 -> 27.9 mm
- net Net-(Q1-D): track 15.3 -> 0.00 mm
- net /Q1-D: track 0.00 -> 15.3 mm
- net /VCC: track 34.5 -> 45.3 mm
- net Net-(D1-A): track 42.4 -> 31.8 mm, vias 0 -> 2
- net Net-(U1-FB): track 13.2 -> 20.2 mm, vias 0 -> 2
- net Net-(J1-Pin_2): track 22.1 -> 16.2 mm
- net /Q1-S: track 17.7 -> 20.5 mm
- net Net-(R8-Pad1): track 2.07 -> 4.25 mm
- net Net-(D2-A): track 8.76 -> 10.6 mm
- net Net-(U1-VREF): track 26.6 -> 27.3 mm
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- removed copper zone on F.Cu, net +12V
