File: DC-DC 12-450V.kicad_sch (KiCad schematic)
At the start: 34 parts, among them J1 12V input, J2 HV output, Q1 IRF3205, Q2 S8050, U1 UC3843_DIP8

Commit message: Add files via upload
Parts:
- D2: value FES8JT -> MUR860
- R11: value 15mR -> 0.015R
- U1: value UC3843_DIP8 -> UC3843BN_DIP8
Changed lines of the file:
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@@
 			)
 		)
-		(property "Value" "FES8JT"
+		(property "Value" "MUR860"
 			(at 217.17 67.31 0)
 			(effects
@@
 			)
 		)
-		(property "Value" "UC3843_DIP8"
+		(property "Value" "UC3843BN_DIP8"
 			(at 148.1933 88.9 0)
 			(effects
@@
 			)
 		)
-		(property "Value" "15mR"
+		(property "Value" "0.015R"
 			(at 188.214 113.538 0)
 			(effects

Commit message: Add files via upload
Parts:
- removed TP1: Q1-D, TestPoint:TestPoint_THTPad_D3.0mm_Drill1.5mm, symbol Connector:TestPoint
- removed TP2, TP3: +12V, TestPoint:TestPoint_THTPad_D3.0mm_Drill1.5mm, symbol Connector:TestPoint
- removed TP4: HV_D-A, TestPoint:TestPoint_THTPad_D3.0mm_Drill1.5mm, symbol Connector:TestPoint
- added TR1: ~, symbol Transformer:TEZ10.0-D-1
- C6, C7, D2, J1, J2, Q1, RV1, U1: now left out of the parts list
- R11: value 0.015R -> 0.015R/3W; footprint Resistor_SMD:R_2816_7142Metric -> Resistor_SMD:R_2512_6332Metric; now left out of the parts list
Connections:
- net +12V: now also TR1.1, TR1.11
- net D2-A: now reaches D2.2 (A)
- net D2-A: now also TR1.8
- net Q1-S: now reaches Q1.3 (S), R11.1, R4.2
- net Q1-D: now reaches Q1.2 (D)
- net Q1-D: now also TR1.6
Other:
- moved on the sheet: D2
