File: DC-DC 12-450V.kicad_sch (KiCad schematic)
At the start: 33 parts, among them J1 12V input, J2 HV output, Q1 IRF3205, Q2 S8050, U1 UC3843BN_DIP8

Commit message: Add files via upload
Parts:
- RV1: footprint Potentiometer_THT:Potentiometer_Bourns_3266Y_Vertical -> Potentiometer_THT:Potentiometer_Bourns_3296W_Vertical
Changed lines of the file:
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@@
 			)
 		)
-		(property "Footprint" "Potentiometer_THT:Potentiometer_Bourns_3266Y_Vertical"
+		(property "Footprint" "Potentiometer_THT:Potentiometer_Bourns_3296W_Vertical"
 			(at 170.18 54.61 0)
 			(effects

Commit message: Add files via upload
Parts:
- removed D4: PESD12VL1BA, Diode_SMD:D_SOD-323, symbol Diode:SD12_SOD323
- added C9: 100u/35V, Capacitor_THT:CP_Radial_D7.5mm_P2.50mm, symbol Device:C_Polarized
- added JP1: SolderJumper_2_Open, Jumper:SolderJumper-2_P1.3mm_Open_Pad1.0x1.5mm, symbol Jumper:SolderJumper_2_Open
- C7: value 1500u/16V -> 1000u/35V
- D2: value MUR860 -> UF5407-8; footprint Package_TO_SOT_THT:TO-220-2_Vertical -> Diode_THT:D_DO-201AD_P15.24mm_Horizontal; symbol Device:D_Filled -> Diode:UF5407; now in the parts list
- F2: value 1.5A/13.2V -> 1.5A/24V; footprint Fuse:Fuse_1206_3216Metric_Pad1.42x1.75mm_HandSolder -> Fuse:Fuse_1812_4532Metric_Pad1.30x3.40mm_HandSolder
- J1: value 12V input -> 12~24V input
- R12: value 1K -> 2K2
- TR1: value ~ -> EC2828; now in the parts list
Connections:
- net GND: now also C9.2, JP1.2 (B)
- net Q1-D: now also TR1.11
- net Q1-S: now also JP1.1 (A)
- net VCC: now also C9.1
- net +12V renamed +12~24V
- net +12~24V: no longer TR1.11
