File: V2.0/DC-DC 12-450V V2.kicad_sch (KiCad schematic)
At the start: 36 parts, among them J1 12V input, J2 HV output, Q1 IRF3205, Q2 S8050, Q3 IRF3205, U1 UC3843BN_DIP8

Commit message: Add files via upload
Parts:
- added JP1, JP2: SolderJumper_2_Open, Jumper:SolderJumper-2_P1.3mm_Open_Pad1.0x1.5mm, symbol Jumper:SolderJumper_2_Open
- C7: value 1000u/16V -> 1000u/35V
- C9: value 100u/16V -> 100u/35V
- D2: value MUR860 -> UF5407-8; footprint Package_TO_SOT_THT:TO-220-2_Vertical -> Diode_THT:D_DO-201AD_P15.24mm_Horizontal; symbol Device:D_Filled -> Diode:UF5407; now in the parts list
- F2: value 1.5A/13.2V -> 1.5A/24V; footprint Fuse:Fuse_1206_3216Metric_Pad1.42x1.75mm_HandSolder -> Fuse:Fuse_1812_4532Metric_Pad1.30x3.40mm_HandSolder
- J1: value 12V input -> 12~24V input
- R12: value 1K -> 2K2
Connections:
- net +12V: no longer C7.1, F2.1, R12.2, R13.1, TR1.1
- net GND: now also JP1.2 (B)
- net Q1-S: now also JP1.1 (A)
- net VCC: now also JP2.2 (B)
- new net +12~24V: C7.1, F2.1, JP2.1 (A), R12.2, R13.1, TR1.1
