File: V2.0/DC-DC 12-450V V2.kicad_pcb (KiCad board)
At the start: 2 copper layers, 85 x 50 mm, 49 parts, among them J1 12V input, J2 HV output, Q1 IRF3205, Q2 S8050, Q3 IRF3205, U1 UC3843BN_DIP8

Commit message: Add files via upload
Parts:
- moved C7 62.8 mm to (128.4, 98.0)
- moved D1 8.28 mm to (109.5, 100.0)
Routing:
- net Net-(D1-A): track 51.3 -> 43.8 mm
- net +12V: track 94.1 -> 91.2 mm
Changed lines of the file:
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@@
 	(title_block
 		(title "DC-DC 12V > 200~450V")
-		(date "2026-02-05")
+		(date "2026-02-07")
 		(rev "V2.0")
 		(company "Z32IT")
@@
 	(footprint "Capacitor_THT:CP_Radial_D10.0mm_P5.00mm"
 		(layer "F.Cu")
-		(at 180.617677 63.25 180)
+		(at 128.367677 98 180)
 		(descr "CP, Radial series, Radial, pin pitch=5.00mm, , diameter=10mm, Electrolytic Capacitor")
 		(tags "CP Radial series Radial pin pitch 5.00mm  diameter 10mm Electrolytic Capacitor")
@@
 			(size 3 3)
 			(drill 1)
-			(layers)
+			(layers "*.Cu")
 			(remove_unused_layers no)
 		)
@@
 		(tags "resistor")
 		(property "Reference" "R7"
-			(at 0 2 0)
+			(at 3.25 0 0)
 			(layer "F.SilkS")
 			(effects
@@
 			(size 3 3)
 			(drill 1)
-			(layers)
+			(layers "*.Cu")
 			(remove_unused_layers no)
 		)
@@
 			(size 3 3)
 			(drill 1)
-			(layers)
+			(layers "*.Cu")
 			(remove_unused_layers no)
 		)
@@
 			(size 3 3)
 			(drill 1)
-			(layers)
+			(layers "*.Cu")
 			(remove_unused_layers no)
 			(pinfunction "1")
@@
 		(tags "resistor")
 		(property "Reference" "R6"
-			(at 0 1.75 0)
+			(at -3.25 0 0)
 			(layer "F.SilkS")
 			(effects
@@
 	(footprint "LED_SMD:LED_1206_3216Metric"
 		(layer "F.Cu")
-		(at 117.75 100.75 180)
+		(at 109.5 100 180)
 		(descr "LED SMD 1206 (3216 Metric), square (rectangular) end terminal, IPC_7351 nominal, (Body size source: http://www.tortai-tech.com/upload/download/2011102023233369053.pdf), generated with kicad-footprint-generator")
 		(tags "LED")
@@
 	)
 	(gr_text "+"
-		(at 174.75 100 0)
+		(at 174.75 100.5 0)
 		(layer "F.SilkS")
 		(effects
@@
 	)
 	(segment
-		(start 110.5375 100.75)
-		(end 116.35 100.75)
-		(width 0.5)
-		(layer "F.Cu")
-		(net 7)
-	)
-	(segment
 		(start 115.525 74.7625)
 		(end 115.45 74.6875)
@@
 	)
 	(segment
+		(start 105.0375 96.9375)
+		(end 108.1 100)
+		(width 0.5)
+		(layer "F.Cu")
+		(net 7)
+	)
+	(segment
+		(start 105.0375 95.25)
+		(end 105.0375 96.9375)
+		(width 0.5)
+		(layer "F.Cu")
+		(net 7)
+	)
+	(segment
 		(start 102.25 85.4625)
 		(end 102.25 92.4625)
@@
 	)
 	(segment
-		(start 105.0375 95.25)
-		(end 110.5375 100.75)
-		(width 0.5)
-		(layer "F.Cu")
-		(net 7)
-	)
-	(segment
 		(start 100.5375 83.75)
 		(end 100.5375 79.25)
@@
 	)
 	(segment
+		(start 135.75 91.25)
+		(end 135.117677 91.25)
+		(width 1.5)
+		(layer "F.Cu")
+		(net 9)
+	)
+	(segment
 		(start 160.5 66.7125)
 		(end 160.5 71)
@@
 	)
 	(segment
-		(start 180.617677 63.25)
-		(end 180.617677 75.882323)
-		(width 2)
-		(layer "F.Cu")
-		(net 9)
-	)
-	(segment
 		(start 180.617677 75.882323)
 		(end 180.25 76.25)
@@
 	)
 	(segment
+		(start 135.117677 91.25)
+		(end 128.367677 98)
+		(width 2)
+		(layer "F.Cu")
+		(net 9)
+	)
+	(segment
 		(start 160.75 73.0875)
 		(end 160.75 71.25)
@@
 	)
 	(segment
-		(start 180.25 63.617677)
-		(end 180.617677 63.25)
-		(width 0.2)
-		(layer "F.Cu")
-		(net 9)
-	)
-	(segment
 		(start 150.75 76.25)
 		(end 135.75 91.25)
@@
 		(polygon
 			(pts
-				(xy 98.5 57.75) (xy 98.5 73) (xy 111 73) (xy 111 79) (xy 110.75 79) (xy 104.75 79) (xy 104.75 102.5)
-				(xy 142.5 102.5) (xy 142.5 89) (xy 183.5 89) (xy 183.5 57.75)
+				(xy 98.5 57.75) (xy 98.5 73) (xy 111 73) (xy 111 79) (xy 110.75 79) (xy 104.75 79) (xy 104.75 103.25)
+				(xy 142.5 103.25) (xy 142.5 89) (xy 183.5 89) (xy 183.5 57.75)
 			)
 		)

Commit message: Add files via upload
Parts:
- added JP1: SolderJumper_2_Open, Jumper:SolderJumper-2_P1.3mm_Open_Pad1.0x1.5mm, F.Cu at (138.5, 64.7)
- added JP2: SolderJumper_2_Open, Jumper:SolderJumper-2_P1.3mm_Open_Pad1.0x1.5mm, F.Cu at (132.2, 87.2)
- C7: value 1000u/16V -> 1000u/35V
- C9: value 100u/16V -> 100u/35V
- D2: value MUR860 -> UF5407-8; footprint Package_TO_SOT_THT:TO-220-2_Vertical -> Diode_THT:D_DO-201AD_P15.24mm_Horizontal
- F2: value 1.5A/13.2V -> 1.5A/24V; footprint Fuse:Fuse_1206_3216Metric_Pad1.42x1.75mm_HandSolder -> Fuse:Fuse_1812_4532Metric_Pad1.30x3.40mm_HandSolder
- J1: value 12V input -> 12~24V input
- R12: value 1K -> 2K2
- moved R4 27.8 mm to (121.5, 60.9), turned to 0 degrees
- moved R2 17.7 mm to (116.2, 94.2), turned to 180 degrees
- moved F2 12.2 mm to (141.2, 88.8), turned to 90 degrees
- moved R3 9.91 mm to (116.2, 97.0), turned to 180 degrees
- moved C3 5.63 mm to (108.0, 94.2), turned to 0 degrees
- moved C8 5.50 mm to (126.8, 81.5)
- moved D2 4.27 mm to (171.8, 105.0)
- moved C6 1.52 mm to (171.0, 97.9), turned to 90 degrees
- moved D1 0.75 mm to (109.5, 99.2), turned to 0 degrees
- moved R8 0.50 mm to (149.8, 94.8)
- moved R9 0.50 mm to (149.8, 102.5)
Connections:
- C7 pad 1: +12V -> +12~24V
- F2 pad 1: +12V -> +12~24V
- PAD2 pad 2: +12V -> +12~24V
- PAD3 pad 3: +12V -> /VCC
- PAD7 pad 7: +12V -> +12~24V
- PAD8 pad 8: +12V -> +12~24V
- Q1 pad 2: Net-(Q1-D) -> /Q1-D
- R12 pad 2: +12V -> +12~24V
- R13 pad 1: +12V -> +12~24V
Routing:
- net +12~24V: track 0.00 -> 93.9 mm
- net +12V: track 91.2 -> 0.00 mm
- net Net-(U1-CS): track 78.6 -> 39.9 mm, vias 3 -> 4
- net /Q1-S: track 9.65 -> 27.9 mm
- net Net-(D1-A): track 43.8 -> 31.0 mm, vias 0 -> 2
- net /VCC: track 37.6 -> 48.3 mm
- net GND: track 27.2 -> 19.4 mm, vias 31 -> 38
- net Net-(U1-FB): track 13.2 -> 20.5 mm, vias 0 -> 2
- net Net-(D2-K): track 46.3 -> 41.0 mm
- net Net-(D2-A): track 8.76 -> 10.5 mm
- net Net-(R9-Pad1): track 82.2 -> 84.0 mm, vias 4 -> 0

Commit message: Add files via upload
Changed lines of the file:
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@@
 	(title_block
 		(title "DC-DC 12~24V > 200~450V")
-		(date "2026-02-08")
+		(date "2026-02-09")
 		(rev "V2.1")
 		(company "Z32IT")
@@
 		(end 138.5 61.155)
 		(width 1.5)
-		(layer "F.Cu")
+		(layers "F.Cu" "F.Mask")
+		(solder_mask_margin 0)
 		(net 18)
 	)
@@
 		(end 144.9075 60.945)
 		(width 2)
-		(layer "F.Cu")
+		(layers "F.Cu" "F.Mask")
+		(solder_mask_margin 0)
 		(net 18)
 	)
@@
 	)
 	(zone
+		(net 0)
+		(net_name "")
+		(layers "F.Cu" "B.Cu")
+		(hatch edge 0.5)
+		(connect_pads
+			(clearance 0)
+		)
+		(min_thickness 0.25)
+		(filled_areas_thickness no)
+		(keepout
+			(tracks not_allowed)
+			(vias not_allowed)
+			(pads not_allowed)
+			(copperpour not_allowed)
+			(footprints allowed)
+		)
+		(placement
+			(enabled no)
+			(sheetname "")
+		)
+		(fill
+			(thermal_gap 0.5)
+			(thermal_bridge_width 0.5)
+		)
+		(polygon
+			(pts
+				(xy 161.25 59.25) (xy 161.25 62.5) (xy 167.75 62.5) (xy 167.75 59.25)
+			)
+		)
+	)
+	(zone
 		(net 4)
 		(net_name "GND")
@@
 			)
 		)
+	)
+	(zone
+		(net 0)
+		(net_name "")
+		(layers "F.Cu" "B.Cu")
+		(hatch edge 0.5)
+		(connect_pads
+			(clearance 0)
+		)
+		(min_thickness 0.25)
+		(filled_areas_thickness no)
+		(keepout
+			(tracks not_allowed)
+			(vias not_allowed)
+			(pads not_allowed)
+			(copperpour not_allowed)
+			(footprints allowed)
+		)
+		(placement
+			(enabled no)
+			(sheetname "")
+		)
+		(fill
+			(thermal_gap 0.5)
+			(thermal_bridge_width 0.5)
+		)
+		(polygon
+			(pts
+				(xy 130.75 58.25) (xy 130.75 62.5) (xy 137.5 62.5) (xy 137.5 63.25) (xy 142.5 63.25) (xy 142.5 58.25)
+			)
+		)
